File: Kicad/DC Electronic Load.kicad_sch (KiCad schematic)
At the start: 33 parts

Commit message: Completed more of the schmatic
Parts:
- added J?: Screw_Terminal_01x02, symbol Connector:Screw_Terminal_01x02
- added R? (x2): R, symbol Device:R
- added RV?: 10k, symbol Device:R_Potentiometer
Connections:
- net 5V REF: now also RV?.1
- net GND: now also J?.2 (Pin_2), R?.1, RV?.3
- net Gate1: now also U?.1
- net Gate2: now also U?.7
- net at U?.12 (+): now also R?.1, R?.2
- net Voltage_Sense: now reaches U?.13 (-)
- net Voltage_Sense: now also U?.14
- net Vin: now reaches Q?.2 (D), Q?.2 (D)
- net Vin: now also J?.1 (Pin_1), R?.2
- net Curr_Sense_1: now reaches Q?.3 (S), R?.1
- net Curr_Sense_1: now also U?.2 (-)
- net CURRENT_SETPOINT: now reaches U?.5 (+)
- net CURRENT_SETPOINT: now also U?.3 (+), RV?.2
- net Curr_Sense_2: now reaches U?.6 (-)
- net Curr_Sense_2: now also Q?.3 (S), R?.1
Other:
- moved on the sheet: HS?, TH?, U?A, U?B, U?C, U?D
